File: bio-power-2.kicad_pcb (KiCad board)
At the start: 4 copper layers, 31 x 24 mm, 33 parts, among them J1 TYPE-C-31-M-12, J2 6vdc, J3 TC2030-IDC, U1 STUSB4500QTR, U3 LT3041ADE-PBF

Commit message: finish
Routing:
- net GND: track 13.8 -> 28.5 mm, vias 29 -> 31
- net Net-(D1-A): track 49.8 -> 51.5 mm
Other:
- board size 31 x 24 mm -> 32.5 x 24 mm
Changed lines of the file:
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@@
 			(unlocked yes)
 			(layer "F.SilkS")
+			(hide yes)
 			(effects
 				(font
@@
 			)
 		)
-		(property "Footprint" "05-08-1708_ADI"
+		(property "Footprint" "lt3041:05-08-1708_ADI"
 			(at 0 0 -90)
 			(unlocked yes)
@@
 			(at 0 -1.448 0)
 			(layer "F.SilkS")
+			(hide yes)
 			(effects
 				(font
@@
 			(unlocked yes)
 			(layer "F.SilkS")
+			(hide yes)
 			(effects
 				(font
@@
 			(layer "F.Fab")
 		)
-		(fp_text user "*"
-			(at -1.36525 -2.1994 180)
-			(layer "F.SilkS")
-			(effects
-				(font
-					(size 1 1)
-					(thickness 0.15)
-				)
-			)
-		)
-		(fp_text user "*"
-			(at -1.36525 -2.1994 180)
-			(unlocked yes)
-			(layer "F.SilkS")
-			(effects
-				(font
-					(size 1 1)
-					(thickness 0.15)
-				)
-			)
-		)
-		(fp_text user "*"
-			(at -0.4191 -1.1072 180)
-			(layer "F.Fab")
-			(effects
-				(font
-					(size 1 1)
-					(thickness 0.15)
-				)
-			)
-		)
 		(fp_text user "${REFERENCE}"
 			(at 0 0 180)
@@
 			)
 		)
-		(fp_text user "*"
-			(at -0.4191 -1.1072 180)
-			(unlocked yes)
-			(layer "F.Fab")
-			(effects
-				(font
-					(size 1 1)
-					(thickness 0.15)
-				)
-			)
-		)
 		(pad "1" smd rect
 			(at -1.11125 -0.649999 180)
@@
 			(at -2.75 0.265 180)
 			(layer "F.SilkS")
+			(hide yes)
 			(effects
 				(font
@@
 			(at 0 -1.43 0)
 			(layer "F.SilkS")
+			(hide yes)
 			(effects
 				(font
@@
 			(at 0 -3.5 0)
 			(layer "F.SilkS")
+			(hide yes)
 			(effects
 				(font
@@
 	)
 	(gr_rect
-		(start 82 65)
+		(start 80.5 65)
 		(end 113 89)
 		(stroke
@@
 	)
 	(segment
+		(start 97.5225 79.79)
+		(end 96.725 79.79)
+		(width 0.25)
+		(layer "F.Cu")
+		(net 1)
+	)
+	(segment
 		(start 103.25 79.1978)
 		(end 103.25 77.75)
@@
 	(segment
 		(start 97.4125 79.79)
-		(end 96.725 79.79)
+		(end 97.3025 79.79)
 		(width 0.25)
 		(layer "F.Cu")
@@
 	)
 	(segment
+		(start 97.65 79.9)
+		(end 97.5225 79.79)
+		(width 0.25)
+		(layer "F.Cu")
+		(net 1)
+	)
+	(segment
+		(start 97.3025 79.79)
+		(end 97.65 79.9)
+		(width 0.25)
+		(layer "F.Cu")
+		(net 1)
+	)
+	(segment
 		(start 102.564399 77.75)
 		(end 103.25 77.75)
@@
 	)
 	(via
+		(at 97.65 79.9)
+		(size 0.6)
+		(drill 0.3)
+		(layers "F.Cu" "B.Cu")
+		(net 1)
+	)
+	(via
 		(at 104.25 78)
 		(size 0.6)
@@
 	)
 	(via
-		(at 88.25 73.75)
+		(at 88.25 74.05)
 		(size 0.6)
 		(drill 0.3)
@@
 	)
 	(via
+		(at 98.45 78.85)
+		(size 0.6)
+		(drill 0.3)
+		(layers "F.Cu" "B.Cu")
+		(free yes)
+		(net 1)
+	)
+	(via
 		(at 101.5 80.75)
 		(size 0.6)
@@
 	)
 	(segment
+		(start 94.7 77.765)
+		(end 94.7 79.315)
+		(width 0.2)
+		(layer "In2.Cu")
+		(net 1)
+	)
+	(segment
+		(start 97.365 77.765)
+		(end 98.45 78.85)
+		(width 0.2)
+		(layer "In2.Cu")
+		(net 1)
+	)
+	(segment
+		(start 96.25 77.765)
+		(end 94.7 77.765)
+		(width 0.2)
+		(layer "In2.Cu")
+		(net 1)
+	)
+	(segment
+		(start 96.25 77.765)
+		(end 96.25 79.315)
+		(width 0.2)
+		(layer "In2.Cu")
+		(net 1)
+	)
+	(segment
+		(start 96.25 77.765)
+		(end 97.365 77.765)
+		(width 0.2)
+		(layer "In2.Cu")
+		(net 1)
+	)
+	(segment
+		(start 96.29 78.54)
+		(end 97.65 79.9)
+		(width 0.2)
+		(layer "In2.Cu")
+		(net 1)
+	)
+	(segment
+		(start 95.475 79.315)
+		(end 95.475 77.765)
+		(width 0.2)
+		(layer "In2.Cu")
+		(net 1)
+	)
+	(segment
+		(start 94.7 79.315)
+		(end 96.25 79.315)
+		(width 0.2)
+		(layer "In2.Cu")
+		(net 1)
+	)
+	(segment
+		(start 96.25 78.54)
+		(end 96.29 78.54)
+		(width 0.2)
+		(layer "In2.Cu")
+		(net 1)
+	)
+	(segment
+		(start 94.7 78.54)
+		(end 96.25 78.54)
+		(width 0.2)
+		(layer "In2.Cu")
+		(net 1)
+	)
+	(segment
 		(start 93.3725 73.1775)
 		(end 99.75 73.1775)
@@
 	)
 	(segment
-		(start 98.4063 72.3437)
-		(end 98.5 72.25)
-		(width 0.5)
-		(layer "F.Cu")
-		(net 34)
-	)
-	(segment
-		(start 94.5 72.25)
-		(end 94.5937 72.3437)
-		(width 0.5)
-		(layer "F.Cu")
-		(net 34)
-	)
-	(segment
 		(start 101.925 70.5494)
 		(end 101.925 72.55)
@@
 	)
 	(segment
-		(start 98.8525 72.25)
-		(end 98.5 72.25)
+		(start 99.7975 71.3525)
+		(end 100.6006 70.5494)
+		(width 0.5)
+		(layer "F.Cu")
+		(net 34)
+	)
+	(segment
+		(start 100.6006 70.5494)
+		(end 101.925 70.5494)
 		(width 0.5)
 		(layer "F.Cu")
@@
 	(segment
 		(start 99.75 71.3525)
-		(end 99.75 71.1)
+		(end 99.7975 71.3525)
 		(width 0.5)
 		(layer "F.Cu")
@@
 	)
 	(segment
-		(start 100.8994 70.5494)
-		(end 101.925 70.5494)
-		(width 0.5)
-		(layer "F.Cu")
-		(net 34)
-	)
-	(segment
-		(start 99.75 71.3525)
-		(end 98.8525 72.25)
-		(width 0.5)
-		(layer "F.Cu")
-		(net 34)
-	)
-	(segment
 		(start 92.25 76.5)
 		(end 94.0825 76.46)
@@
 	)
 	(segment
-		(start 100.6 70.25)
-		(end 100.8994 70.5494)
+		(start 94.5937 72.3437)
+		(end 98.7588 72.3437)
 		(width 0.5)
 		(layer "F.Cu")
@@
 	)
 	(segment
+		(start 94.5 72.25)
+		(end 94.5937 72.3437)
+		(width 0.5)
+		(layer "F.Cu")
+		(net 34)
+	)
+	(segment
 		(start 99.85 71.35)
 		(end 99.75 71.5)
@@
 	)
 	(segment
-		(start 94.5937 72.3437)
-		(end 98.4063 72.3437)
-		(width 0.5)
-		(layer "F.Cu")
-		(net 34)
-	)
-	(segment
 		(start 88.1 79.475)
 		(end 88.275 79.65)
@@
 	)
 	(segment
-		(start 99.75 71.1)
-		(end 100.6 70.25)
+		(start 98.7588 72.3437)
+		(end 99.75 71.3525)
 		(width 0.5)
 		(layer "F.Cu")
@@
 	)
 	(segment
-		(start 89.9 82.460661)
-		(end 89.9 79.65)
+		(start 89.9 79.65)
+		(end 88.3 79.65)
 		(width 0.5)
 		(layer "B.Cu")
@@
 	)
 	(segment
-		(start 91.439339 84)
-		(end 89.9 82.460661)
+		(start 95.5 82.524616)
+		(end 95.5 84.1)
 		(width 0.5)
 		(layer "B.Cu")
@@
 	)
 	(segment
-		(start 95.5 81.565)
-		(end 95.5 84)
+		(start 92.310661 76.5)
+		(end 92.25 76.5)
 		(width 0.5)
 		(layer "B.Cu")
@@
 	)
 	(segment
-		(start 89.9 79.65)
-		(end 88.3 79.65)
+		(start 99.85 71.35)
+		(end 99.85 80.4)
 		(width 0.5)
 		(layer "B.Cu")
@@
 	)
 	(segment
-		(start 92.310661 76.5)
-		(end 92.25 76.5)
+		(start 99.85 80.4)
+		(end 98.9397 81.3103)
 		(width 0.5)
 		(layer "B.Cu")
@@
 	)
 	(segment
-		(start 95.5 84.1)
-		(end 91.439339 84)
+		(start 89.9 83.65)
+		(end 89.9 79.65)
 		(width 0.5)
 		(layer "B.Cu")
@@
 	)
 	(segment
-		(start 95.5 84)
-		(end 95.5 84.1)
+		(start 98.9397 81.3103)
+		(end 96.714316 81.3103)
 		(width 0.5)
 		(layer "B.Cu")
@@
 	)
 	(segment
-		(start 99.85 77.215)
-		(end 95.5 81.565)
+		(start 93 75.810661)
+		(end 92.310661 76.5)
 		(width 0.5)
 		(layer "B.Cu")
@@
 	)
 	(segment
-		(start 93 75.810661)
-		(end 92.310661 76.5)
+		(start 90.35 84.1)
+		(end 89.9 83.65)
 		(width 0.5)
 		(layer "B.Cu")
@@
 	)
 	(segment
-		(start 99.85 71.35)
-		(end 99.85 77.215)
+		(start 95.5 84.1)
+		(end 90.35 84.1)
+		(width 0.5)
+		(layer "B.Cu")
+		(net 34)
+	)
+	(segment
+		(start 96.714316 81.3103)
+		(end 95.5 82.524616)
 		(width 0.5)
 		(layer "B.Cu")

Commit message: pictures add
Connections:
- net Net-(J3-Pin_2) renamed /ALERT
- net Net-(J3-Pin_4) renamed /SDA
- net Net-(J3-Pin_6) renamed /SCL
- J3 pad 1: unconnected-(J3-Pin_1-Pad1) -> GND
- J3 pad 3: unconnected-(J3-Pin_3-Pad3) -> GND
Routing:
- net GND: vias 31 -> 33
